Commit message: Improve phone_to_omx
1. Change robot.urdf to work with lerobot
    Remove unused names,
    end_effector_link -> gripper_frame_link
    joint* -> each joint name in Lerobot
2. id id= omx_follower_phone -> omx_follower_arm, skip calibration, using calibration/omx_follower_arm.jason

File: examples/phone_to_omx/urdf/robot.urdf (robot description, URDF)
Before this commit: robot omx_f, 10 links, 9 joints
Links:
- removed link end_effector_link
- removed link world
- added link gripper_frame_link; visual box size=0.01 0.01 0.01
Joints:
- removed joint gripper_joint_1
- removed joint joint1
- removed joint joint2
- removed joint joint3
- removed joint joint4
- removed joint joint5
- removed joint world_fixed
- added joint elbow_flex: type revolute, parent link2, child link3, origin xyz=0.0415 0 0.11315 rpy=0 0 0, axis 0 1 0, limit lower=-6.283185307179586 upper=6.283185307179586 effort=1000 velocity=4.8
- added joint gripper: type revolute, parent link5, child link6, origin xyz=0.0295 0.0075 0 rpy=0 0 0, axis 0 0 1, limit lower=-6.283185307179586 upper=6.283185307179586 effort=1000 velocity=4.8
- added joint shoulder_lift: type revolute, parent link1, child link2, origin xyz=0 0 0.0635 rpy=0 0 0, axis 0 1 0, limit lower=-6.283185307179586 upper=6.283185307179586 effort=1000 velocity=4.8
- added joint shoulder_pan: type revolute, parent link0, child link1, origin xyz=-0.01125 0 0.034 rpy=0 0 0, axis 0 0 1, limit lower=-6.283185307179586 upper=6.283185307179586 effort=1000 velocity=4.8
- added joint wrist_flex: type revolute, parent link3, child link4, origin xyz=0.162 0 0 rpy=0 0 0, axis 0 1 0, limit lower=-6.283185307179586 upper=6.283185307179586 effort=1000 velocity=4.8
- added joint wrist_roll: type revolute, parent link4, child link5, origin xyz=0.0287 0 0 rpy=0 0 0, axis 1 0 0, limit lower=-6.283185307179586 upper=6.283185307179586 effort=1000 velocity=4.8
- joint end_effector_joint: child end_effector_link -> gripper_frame_link

Commit message: Update URDF, gripper motor change
1. gripper m288 -> m077
2. link? -> same name to SO101
    Add lower_arm_frame_link, lower_arm_frame_joint for android-teleop

File: examples/phone_to_omx/urdf/robot.urdf (robot description, URDF)
Before this commit: robot omx_f, 9 links, 8 joints
Links:
- removed link link0
- removed link link1
- removed link link2
- removed link link3
- removed link link4
- removed link link5
- removed link link6
- removed link link7
- added link base_link, mass 2.238905100e-01; collision mesh filename=assets/follower_01_base.stl scale=0.001 0.001 0.001; visual mesh filename=assets/follower_01_base.stl scale=0.001 0.001 0.001
- added link gripper_gear_link, mass 1.209067700e-02; collision mesh filename=assets/follower_08_gripper_gear.stl scale=0.001 0.001 0.001; visual mesh filename=assets/follower_08_gripper_gear.stl scale=0.001 0.001 0.001
- added link gripper_link, mass 4.381088700e-02; collision mesh filename=assets/follower_06_pan_Revised.stl scale=0.001 0.001 0.001; visual mesh filename=assets/follower_06_pan_Revised.stl scale=0.001 0.001 0.001
- added link gripper_motor_link, mass 1.209067700e-02; collision mesh filename=assets/follower_07_gripper_motorized.stl scale=0.001 0.001 0.001; visual mesh filename=assets/follower_07_gripper_motorized.stl scale=0.001 0.001 0.001
- added link lower_arm_frame_link, mass 1e-9
- added link lower_arm_link, mass 8.375912900e-02; collision mesh filename=assets/follower_04_middle_horizontal.stl scale=0.001 0.001 0.001; visual mesh filename=assets/follower_04_middle_horizontal.stl scale=0.001 0.001 0.001
- added link shoulder_link, mass 6.598704100e-02; collision mesh filename=assets/follower_02_base_tilt_Revised.stl scale=0.001 0.001 0.001; visual mesh filename=assets/follower_02_base_tilt_Revised.stl scale=0.001 0.001 0.001
- added link upper_arm_link, mass 8.722147100e-02; collision mesh filename=assets/follower_03_middle_verticle.stl scale=0.001 0.001 0.001; visual mesh filename=assets/follower_03_middle_verticle.stl scale=0.001 0.001 0.001
- added link wrist_link, mass 2.997506300e-02; collision mesh filename=assets/follower_05_tip.stl scale=0.001 0.001 0.001; visual mesh filename=assets/follower_05_tip.stl scale=0.001 0.001 0.001
Joints:
- removed joint gripper_joint_2
- added joint gripper_joint_1: type revolute, parent gripper_link, child gripper_gear_link, origin xyz=0.0295 -0.0108 0 rpy=0 0 0, axis 0 0 1, limit lower=-6.283185307179586 upper=6.283185307179586 effort=1000 velocity=4.8, mimic joint=gripper_joint_1 multiplier=-1
- added joint lower_arm_frame_joint: type fixed, parent lower_arm_link, child lower_arm_frame_link, origin xyz=-0.1349 0.0052 0.015 rpy=1.5708 0 -1.5708, axis 0 0 0
- joint elbow_flex: child link3 -> lower_arm_link; parent link2 -> upper_arm_link
- joint end_effector_joint: parent link5 -> gripper_link
- joint gripper: child link6 -> gripper_motor_link; parent link5 -> gripper_link
- joint shoulder_lift: child link2 -> upper_arm_link; parent link1 -> shoulder_link
- joint shoulder_pan: child link1 -> shoulder_link; parent link0 -> base_link
- joint wrist_flex: child link4 -> wrist_link; parent link3 -> lower_arm_link
- joint wrist_roll: child link5 -> gripper_link; parent link4 -> wrist_link
