Commit message: Modify rebearm urdf
Change joint name to match SOARM

File: examples/phone_to_rebearm/urdf/robot.urdf (robot description, URDF)
Before this commit: robot rebearm, 8 links, 7 joints
Links:
- removed link link6
- removed link world
- added link gripper_frame_link, mass 1; collision box size=0.045 0.045 0.95; visual mesh filename=assets/URDF_joint6.stl scale=0.005 0.005 0.005
Joints:
- removed joint joint1
- removed joint joint2
- removed joint joint3
- removed joint joint4
- removed joint joint5
- removed joint joint6
- removed joint world_fixed
- added joint elbow_flex: type revolute, parent link2, child link3, origin xyz=0.0 0.0 0.44 rpy=0.0 0.0 0.0, axis 1 0 0, limit lower=-0.78 upper=-2.09 effort=1 velocity=4.8
- added joint gripper: type revolute, parent link5, child gripper_frame_link, origin xyz=0.0 -0.07 0.178 rpy=0.0 0.0 0.0, axis 1 0 0, limit lower=-1.6 upper=-1.04 effort=1 velocity=4.8
- added joint shoulder_lift: type revolute, parent link1, child link2, origin xyz=0.0 0.0 0.19 rpy=0.0 0.0 0.0, limit lower=0.52 upper=-0.105 effort=1 velocity=4.8
- added joint shoulder_pan: type revolute, parent base_link, child link1, origin xyz=0.0 0.0 0.2 rpy=0.0 0.0 0.0, axis 0 0 1, limit lower=-1.57 upper=1.57 effort=1 velocity=4.8
- added joint wrist_flex: type revolute, parent link3, child link4, origin xyz=0.0 -0.001 0.56 rpy=0 0 0, axis 1 0 0, limit lower=-0.87 upper=-2.09 effort=1 velocity=4.8
- added joint wrist_roll: type revolute, parent link4, child link5, origin xyz=0.0 -0.06 0.3 rpy=0.0 0.0 0.0, axis 0 0 1, limit lower=1.5707963267948966 upper=-1.5707963267948966 effort=1 velocity=4.8

Commit message: Working phone_to _rebearm
1. Modify rebearm's robot.urdf
2. Add print into robot_kinematic_processor.py

File: examples/phone_to_rebearm/urdf/robot.urdf (robot description, URDF)
Before this commit: robot rebearm, 7 links, 6 joints
Links:
- removed link base_link
- added link gripper_moving_link, mass 0.210; collision mesh filename=assets/URDF_joint6.stl scale=0.001 0.001 0.001; visual mesh filename=assets/URDF_joint6.stl scale=0.001 0.001 0.001
- added link link0, mass 0.147; collision mesh filename=assets/URDF_joint0.stl scale=0.001 0.001 0.001; visual mesh filename=assets/URDF_joint0.stl scale=0.001 0.001 0.001
- link gripper_frame_link: mass 1 -> 1e-9; geometry 
- link link1: mass 1 -> 0.147; geometry collision mesh filename=assets/URDF_joint1.stl scale=0.001 0.001 0.001; visual mesh filename=assets/URDF_joint1.stl scale=0.001 0.001 0.001
- link link2: mass 1 -> 0.150; geometry collision mesh filename=assets/URDF_joint2.stl scale=0.001 0.001 0.001; visual mesh filename=assets/URDF_joint2.stl scale=0.001 0.001 0.001
- link link3: mass 1 -> 0.210; geometry collision mesh filename=assets/URDF_joint3.stl scale=0.001 0.001 0.001; visual mesh filename=assets/URDF_joint3.stl scale=0.001 0.001 0.001
- link link4: mass 1 -> 0.250; geometry collision mesh filename=assets/URDF_joint4.stl scale=0.001 0.001 0.001; visual mesh filename=assets/URDF_joint4.stl scale=0.001 0.001 0.001
- link link5: mass 1 -> 0.350; geometry collision mesh filename=assets/URDF_joint5.stl scale=0.001 0.001 0.001; visual mesh filename=assets/URDF_joint5.stl scale=0.001 0.001 0.001
Joints:
- added joint gripper_frame_joint: type fixed, parent link5, child gripper_frame_link, origin xyz=-0.0079 -0.000218121 -0.0981274 rpy=0 3.14159 0, axis 0 0 0
- joint elbow_flex: limit lower=-0.78 upper=-2.09 effort=1 velocity=4.8 -> lower=-1.57 upper=1.57 effort=10 velocity=4.8; origin xyz=0.0 0.0 0.44 rpy=0.0 0.0 0.0 -> xyz=0.0 0.0 0.088 rpy=0.0 0.0 0.0
- joint gripper: child gripper_frame_link -> gripper_moving_link; limit lower=-1.6 upper=-1.04 effort=1 velocity=4.8 -> lower=-1.57 upper=1.57 effort=10 velocity=4.8; origin xyz=0.0 -0.07 0.178 rpy=0.0 0.0 0.0 -> xyz=0.0 -0.014 0.0356 rpy=0.0 0.0 0.0
- joint shoulder_lift: limit lower=0.52 upper=-0.105 effort=1 velocity=4.8 -> lower=-1.57 upper=1.57 effort=10 velocity=4.8; origin xyz=0.0 0.0 0.19 rpy=0.0 0.0 0.0 -> xyz=0.0 0.0 0.038 rpy=0.0 0.0 0.0
- joint shoulder_pan: limit lower=-1.57 upper=1.57 effort=1 velocity=4.8 -> lower=-1.57 upper=1.57 effort=10 velocity=4.8; origin xyz=0.0 0.0 0.2 rpy=0.0 0.0 0.0 -> xyz=0.0 0.0 0.04 rpy=0.0 0.0 0.0; parent base_link -> link0
- joint wrist_flex: limit lower=-0.87 upper=-2.09 effort=1 velocity=4.8 -> lower=-1.57 upper=1.57 effort=10 velocity=4.8; origin xyz=0.0 -0.001 0.56 rpy=0 0 0 -> xyz=0.0 -0.0002 0.112 rpy=0 0 0
- joint wrist_roll: limit lower=1.5707963267948966 upper=-1.5707963267948966 effort=1 velocity=4.8 -> lower=-1.57 upper=1.57 effort=10 velocity=4.8; origin xyz=0.0 -0.06 0.3 rpy=0.0 0.0 0.0 -> xyz=0.0 -0.012 0.06 rpy=0.0 0.0 0.0

Commit message: Implement rebearm teleop-android
1. change folder teleop_omx -> teleop_robot
2. remove .key from gitignore
3. remove print rebearm_follower

File: examples/phone_to_rebearm/urdf/robot.urdf (robot description, URDF)
Before this commit: robot rebearm, 8 links, 7 joints
Links:
- removed link link0
- removed link link1
- removed link link2
- removed link link3
- removed link link4
- removed link link5
- added link base_link, mass 0.147; collision mesh filename=assets/URDF_joint0.stl scale=0.001 0.001 0.001; visual mesh filename=assets/URDF_joint0.stl scale=0.001 0.001 0.001
- added link gripper_link, mass 0.350; collision mesh filename=assets/URDF_joint5.stl scale=0.001 0.001 0.001; visual mesh filename=assets/URDF_joint5.stl scale=0.001 0.001 0.001
- added link lower_arm_frame_link, mass 1e-9
- added link lower_arm_link, mass 0.210; collision mesh filename=assets/URDF_joint3.stl scale=0.001 0.001 0.001; visual mesh filename=assets/URDF_joint3.stl scale=0.001 0.001 0.001
- added link shoulder_link, mass 0.147; collision mesh filename=assets/URDF_joint1.stl scale=0.001 0.001 0.001; visual mesh filename=assets/URDF_joint1.stl scale=0.001 0.001 0.001
- added link upper_arm_link, mass 0.150; collision mesh filename=assets/URDF_joint2.stl scale=0.001 0.001 0.001; visual mesh filename=assets/URDF_joint2.stl scale=0.001 0.001 0.001
- added link wrist_link, mass 0.250; collision mesh filename=assets/URDF_joint4.stl scale=0.001 0.001 0.001; visual mesh filename=assets/URDF_joint4.stl scale=0.001 0.001 0.001
Joints:
- added joint lower_arm_frame_joint: type fixed, parent lower_arm_link, child lower_arm_frame_link, origin xyz=-0.1349 0.0052 0.015 rpy=1.5708 0 -1.5708, axis 0 0 0
- joint elbow_flex: child link3 -> lower_arm_link; parent link2 -> upper_arm_link
- joint gripper: parent link5 -> gripper_link
- joint gripper_frame_joint: parent link5 -> gripper_link
- joint shoulder_lift: child link2 -> upper_arm_link; parent link1 -> shoulder_link
- joint shoulder_pan: child link1 -> shoulder_link; parent link0 -> base_link
- joint wrist_flex: child link4 -> wrist_link; parent link3 -> lower_arm_link
- joint wrist_roll: child link5 -> gripper_link; parent link4 -> wrist_link
